File: Hardware/KiCAD/Indication.sch (KiCad schematic (older format))
At the start: 0 parts

Commit message: more work on PTWS schematic
Parts:
- added D? (x5): LED, symbol LED
- added Q? (x5): 2N7002, symbol 2N7002
- added R? (x5): R, symbol R
Connections:
- new net: D?.1 (K), Q?.3 (D) (x5)
- new net: D?.2 (A), R?.2 (x5)
- new net +3.3V: R?.1, R?.1, R?.1, R?.1, R?.1
- new net 1PPS: Q?.1 (G)
- new net ACTIV_LED: Q?.1 (G)
- new net CONN_LED: Q?.1 (G)
- new net EVENT_LED: Q?.1 (G)
- new net FIX: Q?.1 (G)
- new net GND: Q?.2 (S), Q?.2 (S), Q?.2 (S), Q?.2 (S), Q?.2 (S)

Commit message: More work on PTWS
Parts:
- gave numbers to parts that had none: 15
Changed lines of the file:
@@
 LIBS:Relays
 LIBS:Transistors-BJH
-LIBS:MemoryDevices-BJH
 LIBS:ptws-cache
 EELAYER 25 0
@@
 $EndDescr
 $Comp
-L 2N7002 Q?
+L 2N7002 Q1
 U 1 1 57C32A1D
 P 1200 2100
-F 0 "Q?" H 1400 2175 50  0000 L CNN
+F 0 "Q1" H 1400 2175 50  0000 L CNN
 F 1 "2N7002" H 900 2300 50  0000 L CNN
 F 2 "" H 1400 2025 50  0000 L CIN
@@
 	800  2150 1000 2150
 $Comp
-L +3.3V_BJH #PWR?
+L +3.3V_BJH #PWR027
 U 1 1 57C32A6B
 P 1300 850
-F 0 "#PWR?" H 1300 1040 20  0001 C CNN
+F 0 "#PWR027" H 1300 1040 20  0001 C CNN
 F 1 "+3.3V_BJH" H 1300 1040 51  0001 C CNN
 F 2 "" H 1300 850 60  0001 C CNN
@@
 $EndComp
 $Comp
-L LED D?
+L LED D2
 U 1 1 57C32A8D
 P 1300 1600
-F 0 "D?" H 1300 1700 50  0000 C CNN
+F 0 "D2" H 1300 1700 50  0000 C CNN
 F 1 "LED" H 1300 1500 50  0000 C CNN
 F 2 "" H 1300 1600 50  0000 C CNN
@@
 $EndComp
 $Comp
-L R R?
+L R R11
 U 1 1 57C32AC4
 P 1300 1150
-F 0 "R?" V 1380 1150 50  0000 C CNN
+F 0 "R11" V 1380 1150 50  0000 C CNN
 F 1 "R" V 1300 1150 50  0000 C CNN
 F 2 "" V 1230 1150 50  0000 C CNN
@@
 	1300 900  1300 1000
 $Comp
-L GND #PWR?
+L GND #PWR028
 U 1 1 57C32BC9
 P 1300 2400
-F 0 "#PWR?" H 1300 2150 50  0001 C CNN
+F 0 "#PWR028" H 1300 2150 50  0001 C CNN
 F 1 "GND" H 1300 2250 50  0000 C CNN
 F 2 "" H 1300 2400 50  0000 C CNN
@@
 	1300 2400 1300 2300
 $Comp
-L 2N7002 Q?
+L 2N7002 Q2
 U 1 1 57C32CDA
 P 2500 2100
-F 0 "Q?" H 2700 2175 50  0000 L CNN
+F 0 "Q2" H 2700 2175 50  0000 L CNN
 F 1 "2N7002" H 2200 2300 50  0000 L CNN
 F 2 "" H 2700 2025 50  0000 L CIN
@@
 	2100 2150 2300 2150
 $Comp
-L +3.3V_BJH #PWR?
+L +3.3V_BJH #PWR029
 U 1 1 57C32CE3
 P 2600 850
-F 0 "#PWR?" H 2600 1040 20  0001 C CNN
+F 0 "#PWR029" H 2600 1040 20  0001 C CNN
 F 1 "+3.3V_BJH" H 2600 1040 51  0001 C CNN
 F 2 "" H 2600 850 60  0001 C CNN
@@
 $EndComp
 $Comp
-L LED D?
+L LED D3
 U 1 1 57C32CE9
 P 2600 1600
-F 0 "D?" H 2600 1700 50  0000 C CNN
+F 0 "D3" H 2600 1700 50  0000 C CNN
 F 1 "LED" H 2600 1500 50  0000 C CNN
 F 2 "" H 2600 1600 50  0000 C CNN
@@
 $EndComp
 $Comp
-L R R?
+L R R12
 U 1 1 57C32CEF
 P 2600 1150
-F 0 "R?" V 2680 1150 50  0000 C CNN
+F 0 "R12" V 2680 1150 50  0000 C CNN
 F 1 "R" V 2600 1150 50  0000 C CNN
 F 2 "" V 2530 1150 50  0000 C CNN
@@
 	2600 900  2600 1000
 $Comp
-L GND #PWR?
+L GND #PWR030
 U 1 1 57C32CF8
 P 2600 2400
-F 0 "#PWR?" H 2600 2150 50  0001 C CNN
+F 0 "#PWR030" H 2600 2150 50  0001 C CNN
 F 1 "GND" H 2600 2250 50  0000 C CNN
 F 2 "" H 2600 2400 50  0000 C CNN
@@
 	2600 2400 2600 2300
 $Comp
-L 2N7002 Q?
+L 2N7002 Q3
 U 1 1 57C3315C
 P 3900 2100
-F 0 "Q?" H 4100 2175 50  0000 L CNN
+F 0 "Q3" H 4100 2175 50  0000 L CNN
 F 1 "2N7002" H 3600 2300 50  0000 L CNN
 F 2 "" H 4100 2025 50  0000 L CIN
@@
 	3500 2150 3700 2150
 $Comp
-L +3.3V_BJH #PWR?
+L +3.3V_BJH #PWR031
 U 1 1 57C33165
 P 4000 850
-F 0 "#PWR?" H 4000 1040 20  0001 C CNN
+F 0 "#PWR031" H 4000 1040 20  0001 C CNN
 F 1 "+3.3V_BJH" H 4000 1040 51  0001 C CNN
 F 2 "" H 4000 850 60  0001 C CNN
@@
 $EndComp
 $Comp
-L LED D?
+L LED D4
 U 1 1 57C3316B
 P 4000 1600
-F 0 "D?" H 4000 1700 50  0000 C CNN
+F 0 "D4" H 4000 1700 50  0000 C CNN
 F 1 "LED" H 4000 1500 50  0000 C CNN
 F 2 "" H 4000 1600 50  0000 C CNN
@@
 $EndComp
 $Comp
-L R R?
+L R R13
 U 1 1 57C33171
 P 4000 1150
-F 0 "R?" V 4080 1150 50  0000 C CNN
+F 0 "R13" V 4080 1150 50  0000 C CNN
 F 1 "R" V 4000 1150 50  0000 C CNN
 F 2 "" V 3930 1150 50  0000 C CNN
@@
 	4000 900  4000 1000
 $Comp
-L GND #PWR?
+L GND #PWR032
 U 1 1 57C3317A
 P 4000 2400
-F 0 "#PWR?" H 4000 2150 50  0001 C CNN
+F 0 "#PWR032" H 4000 2150 50  0001 C CNN
 F 1 "GND" H 4000 2250 50  0000 C CNN
 F 2 "" H 4000 2400 50  0000 C CNN
@@
 	4000 2400 4000 2300
 $Comp
-L 2N7002 Q?
+L 2N7002 Q4
 U 1 1 57C33181
 P 5200 2100
-F 0 "Q?" H 5400 2175 50  0000 L CNN
+F 0 "Q4" H 5400 2175 50  0000 L CNN
 F 1 "2N7002" H 4900 2300 50  0000 L CNN
 F 2 "" H 5400 2025 50  0000 L CIN
@@
 	4800 2150 5000 2150
 $Comp
-L +3.3V_BJH #PWR?
+L +3.3V_BJH #PWR033
 U 1 1 57C3318A
 P 5300 850
-F 0 "#PWR?" H 5300 1040 20  0001 C CNN
+F 0 "#PWR033" H 5300 1040 20  0001 C CNN
 F 1 "+3.3V_BJH" H 5300 1040 51  0001 C CNN
 F 2 "" H 5300 850 60  0001 C CNN
@@
 $EndComp
 $Comp
-L LED D?
+L LED D5
 U 1 1 57C33190
 P 5300 1600
-F 0 "D?" H 5300 1700 50  0000 C CNN
+F 0 "D5" H 5300 1700 50  0000 C CNN
 F 1 "LED" H 5300 1500 50  0000 C CNN
 F 2 "" H 5300 1600 50  0000 C CNN
@@
 $EndComp
 $Comp
-L R R?
+L R R14
 U 1 1 57C33196
 P 5300 1150
-F 0 "R?" V 5380 1150 50  0000 C CNN
+F 0 "R14" V 5380 1150 50  0000 C CNN
 F 1 "R" V 5300 1150 50  0000 C CNN
 F 2 "" V 5230 1150 50  0000 C CNN
@@
 	5300 900  5300 1000
 $Comp
-L GND #PWR?
+L GND #PWR034
 U 1 1 57C3319F
 P 5300 2400
-F 0 "#PWR?" H 5300 2150 50  0001 C CNN
+F 0 "#PWR034" H 5300 2150 50  0001 C CNN
 F 1 "GND" H 5300 2250 50  0000 C CNN
 F 2 "" H 5300 2400 50  0000 C CNN
@@
 	5300 2400 5300 2300
 $Comp
-L 2N7002 Q?
+L 2N7002 Q5
 U 1 1 57C3349A
 P 6500 2100
-F 0 "Q?" H 6700 2175 50  0000 L CNN
+F 0 "Q5" H 6700 2175 50  0000 L CNN
 F 1 "2N7002" H 6200 2300 50  0000 L CNN
 F 2 "" H 6700 2025 50  0000 L CIN
@@
 	6100 2150 6300 2150
 $Comp
-L +3.3V_BJH #PWR?
+L +3.3V_BJH #PWR035
 U 1 1 57C334A3
 P 6600 850
-F 0 "#PWR?" H 6600 1040 20  0001 C CNN
+F 0 "#PWR035" H 6600 1040 20  0001 C CNN
 F 1 "+3.3V_BJH" H 6600 1040 51  0001 C CNN
 F 2 "" H 6600 850 60  0001 C CNN
@@
 $EndComp
 $Comp
-L LED D?
+L LED D6
 U 1 1 57C334A9
 P 6600 1600
-F 0 "D?" H 6600 1700 50  0000 C CNN
+F 0 "D6" H 6600 1700 50  0000 C CNN
 F 1 "LED" H 6600 1500 50  0000 C CNN
 F 2 "" H 6600 1600 50  0000 C CNN
@@
 $EndComp
 $Comp
-L R R?
+L R R15
 U 1 1 57C334AF
 P 6600 1150
-F 0 "R?" V 6680 1150 50  0000 C CNN
+F 0 "R15" V 6680 1150 50  0000 C CNN
 F 1 "R" V 6600 1150 50  0000 C CNN
 F 2 "" V 6530 1150 50  0000 C CNN
@@
 	6600 900  6600 1000
 $Comp
-L GND #PWR?
+L GND #PWR036
 U 1 1 57C334B8
 P 6600 2400
-F 0 "#PWR?" H 6600 2150 50  0001 C CNN
+F 0 "#PWR036" H 6600 2150 50  0001 C CNN
 F 1 "GND" H 6600 2250 50  0000 C CNN
 F 2 "" H 6600 2400 50  0000 C CNN

Commit message: More work on PTWS schematic
Parts:
- added C? (x3): C, symbol C
- added Q? (x2): 2N7002, symbol 2N7002
- added R? (x6): R, symbol R
Connections:
- new net: C?.1, C?.2, Q?.1 (G), R?.1, R?.2
- new net: C?.1, Q?.2 (S), Q?.2 (S), R?.2, R?.2
- new net: C?.2, Q?.1 (G), R?.1, R?.2
- new net: R?.1, R?.1, R?.1, R?.1
- new net ALERT1: C?.1, Q?.3 (D), R?.2
- new net ALERT2: C?.2, Q?.3 (D), R?.2
Changed lines of the file:
@@
 Text GLabel 800  2150 0    60   Input ~ 0
 FIX
-Wire Wire Line
-	800  2150 1000 2150
 $Comp
 L +3.3V_BJH #PWR027
@@
 	1    0    0    -1
 $EndComp
-Wire Wire Line
-	1300 1800 1300 1900
-Wire Wire Line
-	1300 1300 1300 1400
-Wire Wire Line
-	1300 900  1300 1000
 $Comp
 L GND #PWR028
@@
 	1    0    0    -1
 $EndComp
-Wire Wire Line
-	1300 2400 1300 2300
 $Comp
 L 2N7002 Q2
@@
 Text GLabel 2100 2150 0    60   Input ~ 0
 1PPS
-Wire Wire Line
-	2100 2150 2300 2150
 $Comp
 L +3.3V_BJH #PWR029
@@
 	1    0    0    -1
 $EndComp
-Wire Wire Line
-	2600 1800 2600 1900
-Wire Wire Line
-	2600 1300 2600 1400
-Wire Wire Line
-	2600 900  2600 1000
 $Comp
 L GND #PWR030
@@
 	1    0    0    -1
 $EndComp
-Wire Wire Line
-	2600 2400 2600 2300
 $Comp
 L 2N7002 Q3
@@
 Text GLabel 3500 2150 0    60   Input ~ 0
 CONN_LED
-Wire Wire Line
-	3500 2150 3700 2150
 $Comp
 L +3.3V_BJH #PWR031
@@
 	1    0    0    -1
 $EndComp
-Wire Wire Line
-	4000 1800 4000 1900
-Wire Wire Line
-	4000 1300 4000 1400
-Wire Wire Line
-	4000 900  4000 1000
 $Comp
 L GND #PWR032
@@
 	1    0    0    -1
 $EndComp
-Wire Wire Line
-	4000 2400 4000 2300
 $Comp
 L 2N7002 Q4
@@
 Text GLabel 4800 2150 0    60   Input ~ 0
 EVENT_LED
-Wire Wire Line
-	4800 2150 5000 2150
 $Comp
 L +3.3V_BJH #PWR033
@@
 	1    0    0    -1
 $EndComp
-Wire Wire Line
-	5300 1800 5300 1900
-Wire Wire Line
-	5300 1300 5300 1400
-Wire Wire Line
-	5300 900  5300 1000
 $Comp
 L GND #PWR034
@@
 	1    0    0    -1
 $EndComp
-Wire Wire Line
-	5300 2400 5300 2300
 $Comp
 L 2N7002 Q5
@@
 Text GLabel 6100 2150 0    60   Input ~ 0
 ACTIV_LED
-Wire Wire Line
-	6100 2150 6300 2150
 $Comp
 L +3.3V_BJH #PWR035
@@
 	1    0    0    -1
 $EndComp
-Wire Wire Line
-	6600 1800 6600 1900
-Wire Wire Line
-	6600 1300 6600 1400
-Wire Wire Line
-	6600 900  6600 1000
 $Comp
 L GND #PWR036
@@
 	1    0    0    -1
 $EndComp
+$Comp
+L 2N7002 Q?
+U 1 1 5806E246
+P 2600 4650
+F 0 "Q?" H 2800 4725 50  0000 L CNN
+F 1 "2N7002" H 2300 4850 50  0000 L CNN
+F 2 "" H 2800 4575 50  0000 L CIN
+F 3 "" H 2600 4650 50  0000 L CNN
+	1    2600 4650
+	1    0    0    -1
+$EndComp
+$Comp
+L 2N7002 Q?
+U 1 1 5806E673
+P 1350 4650
+F 0 "Q?" H 1550 4725 50  0000 L CNN
+F 1 "2N7002" H 1050 4850 50  0000 L CNN
+F 2 "" H 1550 4575 50  0000 L CIN
+F 3 "" H 1350 4650 50  0000 L CNN
+	1    1350 4650
+	-1   0    0    -1
+$EndComp
+$Comp
+L R R?
+U 1 1 5806E74A
+P 1250 3650
+F 0 "R?" V 1330 3650 50  0000 C CNN
+F 1 "R" V 1250 3650 50  0000 C CNN
+F 2 "" V 1180 3650 50  0000 C CNN
+F 3 "" H 1250 3650 50  0000 C CNN
+	1    1250 3650
+	1    0    0    -1
+$EndComp
+$Comp
+L R R?
+U 1 1 5806E7DC
+P 1650 3650
+F 0 "R?" V 1730 3650 50  0000 C CNN
+F 1 "R" V 1650 3650 50  0000 C CNN
+F 2 "" V 1580 3650 50  0000 C CNN
+F 3 "" H 1650 3650 50  0000 C CNN
+	1    1650 3650
+	1    0    0    -1
+$EndComp
+$Comp
+L C C?
+U 1 1 5806E856
+P 1950 3950
+F 0 "C?" H 1975 4050 50  0000 L CNN
+F 1 "C" H 1975 3850 50  0000 L CNN
+F 2 "" H 1988 3800 50  0000 C CNN
+F 3 "" H 1950 3950 50  0000 C CNN
+	1    1950 3950
+	0    1    1    0
+$EndComp
+$Comp
+L R R?
+U 1 1 5806E913
+P 2700 3650
+F 0 "R?" V 2780 3650 50  0000 C CNN
+F 1 "R" V 2700 3650 50  0000 C CNN
+F 2 "" V 2630 3650 50  0000 C CNN
+F 3 "" H 2700 3650 50  0000 C CNN
+	1    2700 3650
+	1    0    0    -1
+$EndComp
+$Comp
+L R R?
+U 1 1 5806E9B1
+P 2300 3650
+F 0 "R?" V 2380 3650 50  0000 C CNN
+F 1 "R" V 2300 3650 50  0000 C CNN
+F 2 "" V 2230 3650 50  0000 C CNN
+F 3 "" H 2300 3650 50  0000 C CNN
+	1    2300 3650
+	1    0    0    -1
+$EndComp
+$Comp
+L C C?
+U 1 1 5806EB77
+P 1950 4200
+F 0 "C?" H 1975 4300 50  0000 L CNN
+F 1 "C" H 1975 4100 50  0000 L CNN
+F 2 "" H 1988 4050 50  0000 C CNN
+F 3 "" H 1950 4200 50  0000 C CNN
+	1    1950 4200
+	0    1    1    0
+$EndComp
+$Comp
+L R R?
+U 1 1 5806F01F
+P 1650 4950
+F 0 "R?" V 1730 4950 50  0000 C CNN
+F 1 "R" V 1650 4950 50  0000 C CNN
+F 2 "" V 1580 4950 50  0000 C CNN
+F 3 "" H 1650 4950 50  0000 C CNN
+	1    1650 4950
+	1    0    0    -1
+$EndComp
+$Comp
+L R R?
+U 1 1 5806F0AD
+P 2300 4950
+F 0 "R?" V 2380 4950 50  0000 C CNN
+F 1 "R" V 2300 4950 50  0000 C CNN
+F 2 "" V 2230 4950 50  0000 C CNN
+F 3 "" H 2300 4950 50  0000 C CNN
+	1    2300 4950
+	1    0    0    -1
+$EndComp
+$Comp
+L C C?
+U 1 1 5806F2D0
+P 2100 4950
+F 0 "C?" H 2125 5050 50  0000 L CNN
+F 1 "C" H 2125 4850 50  0000 L CNN
+F 2 "" H 2138 4800 50  0000 C CNN
+F 3 "" H 2100 4950 50  0000 C CNN
+	1    2100 4950
+	-1   0    0    1
+$EndComp
+Text GLabel 2950 3950 2    60   Output ~ 0
+ALERT1
+Wire Wire Line
+	800  2150 1000 2150
+Wire Wire Line
+	1300 1800 1300 1900
+Wire Wire Line
+	1300 1300 1300 1400
+Wire Wire Line
+	1300 900  1300 1000
+Wire Wire Line
+	1300 2400 1300 2300
+Wire Wire Line
+	2100 2150 2300 2150
+Wire Wire Line
+	2600 1800 2600 1900
+Wire Wire Line
+	2600 1300 2600 1400
+Wire Wire Line
+	2600 900  2600 1000
+Wire Wire Line
+	2600 2400 2600 2300
+Wire Wire Line
+	3500 2150 3700 2150
+Wire Wire Line
+	4000 1800 4000 1900
+Wire Wire Line
+	4000 1300 4000 1400
+Wire Wire Line
+	4000 900  4000 1000
+Wire Wire Line
+	4000 2400 4000 2300
+Wire Wire Line
+	4800 2150 5000 2150
+Wire Wire Line
+	5300 1800 5300 1900
+Wire Wire Line
+	5300 1300 5300 1400
+Wire Wire Line
+	5300 900  5300 1000
+Wire Wire Line
+	5300 2400 5300 2300
+Wire Wire Line
+	6100 2150 6300 2150
+Wire Wire Line
+	6600 1800 6600 1900
+Wire Wire Line
+	6600 1300 6600 1400
+Wire Wire Line
+	6600 900  6600 1000
 Wire Wire Line
 	6600 2400 6600 2300
+Wire Wire Line
+	1250 3800 1250 4450
+Wire Wire Line
+	2700 3800 2700 4450
+Wire Wire Line
+	2300 3800 2300 4800
+Wire Wire Line
+	2100 4700 2400 4700
+Wire Wire Line
+	1650 3800 1650 4800
+Wire Wire Line
+	1650 4700 1550 4700
+Wire Wire Line
+	1800 3950 1650 3950
+Connection ~ 1650 3950
+Wire Wire Line
+	2100 3950 2950 3950
+Connection ~ 2700 3950
+Wire Wire Line
+	2100 4200 2300 4200
+Connection ~ 2300 4200
+Wire Wire Line
+	1800 4200 1250 4200
+Connection ~ 1250 4200
+Wire Wire Line
+	1250 3350 1250 3500
+Wire Wire Line
+	1250 3350 2700 3350
+Wire Wire Line
+	2700 3350 2700 3500
+Wire Wire Line
+	2300 3500 2300 3350
+Connection ~ 2300 3350
+Wire Wire Line
+	1650 3500 1650 3350
+Connection ~ 1650 3350
+Connection ~ 1650 4700
+Connection ~ 2300 4700
+Wire Wire Line
+	2100 4800 2100 4700
+Wire Wire Line
+	2700 4850 2700 5200
+Wire Wire Line
+	2700 5200 1250 5200
+Wire Wire Line
+	1250 5200 1250 4850
+Wire Wire Line
+	1650 5100 1650 5200
+Connection ~ 1650 5200
+Wire Wire Line
+	2100 5100 2100 5200
+Connection ~ 2100 5200
+Wire Wire Line
+	2300 5100 2300 5200
+Connection ~ 2300 5200
+Text GLabel 1000 3950 0    60   Output ~ 0
+ALERT2
+Wire Wire Line
+	1000 3950 1250 3950
+Connection ~ 1250 3950
 $EndSCHEMATC

Commit message: more work on the schematic
Parts:
- removed C?: C, symbol C
- removed R? (x2): R, symbol R
- added R?: R, symbol R
Connections:
- net labels added: +24V_BJH, ALERT
- wire segments 48 -> 50
Other:
- moved on the sheet: C?, Q?, R?
Changed lines of the file:
@@
 LIBS:Relays
 LIBS:Transistors-BJH
+LIBS:MemoryDevices-BJH
 LIBS:ptws-cache
 EELAYER 25 0
@@
 L 2N7002 Q?
 U 1 1 5806E246
-P 2600 4650
-F 0 "Q?" H 2800 4725 50  0000 L CNN
-F 1 "2N7002" H 2300 4850 50  0000 L CNN
-F 2 "" H 2800 4575 50  0000 L CIN
-F 3 "" H 2600 4650 50  0000 L CNN
-	1    2600 4650
+P 2300 4650
+F 0 "Q?" H 2500 4725 50  0000 L CNN
+F 1 "2N7002" H 2500 4650 50  0000 L CNN
+F 2 "" H 2500 4575 50  0000 L CIN
+F 3 "" H 2300 4650 50  0000 L CNN
+	1    2300 4650
 	1    0    0    -1
 $EndComp
@@
 P 1350 4650
 F 0 "Q?" H 1550 4725 50  0000 L CNN
-F 1 "2N7002" H 1050 4850 50  0000 L CNN
+F 1 "2N7002" H 1600 4650 50  0000 L CNN
 F 2 "" H 1550 4575 50  0000 L CIN
 F 3 "" H 1350 4650 50  0000 L CNN
@@
 L R R?
 U 1 1 5806E7DC
-P 1650 3650
-F 0 "R?" V 1730 3650 50  0000 C CNN
-F 1 "R" V 1650 3650 50  0000 C CNN
-F 2 "" V 1580 3650 50  0000 C CNN
-F 3 "" H 1650 3650 50  0000 C CNN
-	1    1650 3650
-	1    0    0    -1
+P 1500 3950
+F 0 "R?" V 1580 3950 50  0000 C CNN
+F 1 "R" V 1500 3950 50  0000 C CNN
+F 2 "" V 1430 3950 50  0000 C CNN
+F 3 "" H 1500 3950 50  0000 C CNN
+	1    1500 3950
+	0    1    1    0
 $EndComp
 $Comp
 L C C?
 U 1 1 5806E856
-P 1950 3950
-F 0 "C?" H 1975 4050 50  0000 L CNN
-F 1 "C" H 1975 3850 50  0000 L CNN
-F 2 "" H 1988 3800 50  0000 C CNN
-F 3 "" H 1950 3950 50  0000 C CNN
-	1    1950 3950
+P 1500 4350
+F 0 "C?" H 1525 4450 50  0000 L CNN
+F 1 "C" H 1525 4250 50  0000 L CNN
+F 2 "" H 1538 4200 50  0000 C CNN
+F 3 "" H 1500 4350 50  0000 C CNN
+	1    1500 4350
 	0    1    1    0
 $EndComp
@@
 L R R?
 U 1 1 5806E913
-P 2700 3650
-F 0 "R?" V 2780 3650 50  0000 C CNN
-F 1 "R" V 2700 3650 50  0000 C CNN
-F 2 "" V 2630 3650 50  0000 C CNN
-F 3 "" H 2700 3650 50  0000 C CNN
-	1    2700 3650
+P 2400 3650
+F 0 "R?" V 2480 3650 50  0000 C CNN
+F 1 "R" V 2400 3650 50  0000 C CNN
+F 2 "" V 2330 3650 50  0000 C CNN
+F 3 "" H 2400 3650 50  0000 C CNN
+	1    2400 3650
 	1    0    0    -1
 $EndComp
@@
 L R R?
 U 1 1 5806E9B1
-P 2300 3650
-F 0 "R?" V 2380 3650 50  0000 C CNN
-F 1 "R" V 2300 3650 50  0000 C CNN
-F 2 "" V 2230 3650 50  0000 C CNN
-F 3 "" H 2300 3650 50  0000 C CNN
-	1    2300 3650
-	1    0    0    -1
+P 2150 3950
+F 0 "R?" V 2230 3950 50  0000 C CNN
+F 1 "R" V 2150 3950 50  0000 C CNN
+F 2 "" V 2080 3950 50  0000 C CNN
+F 3 "" H 2150 3950 50  0000 C CNN
+	1    2150 3950
+	0    1    1    0
 $EndComp
 $Comp
 L C C?
 U 1 1 5806EB77
-P 1950 4200
-F 0 "C?" H 1975 4300 50  0000 L CNN
-F 1 "C" H 1975 4100 50  0000 L CNN
-F 2 "" H 1988 4050 50  0000 C CNN
-F 3 "" H 1950 4200 50  0000 C CNN
-	1    1950 4200
+P 2150 4200
+F 0 "C?" H 2175 4300 50  0000 L CNN
+F 1 "C" H 2175 4100 50  0000 L CNN
+F 2 "" H 2188 4050 50  0000 C CNN
+F 3 "" H 2150 4200 50  0000 C CNN
+	1    2150 4200
 	0    1    1    0
 $EndComp
-$Comp
-L R R?
-U 1 1 5806F01F
-P 1650 4950
-F 0 "R?" V 1730 4950 50  0000 C CNN
-F 1 "R" V 1650 4950 50  0000 C CNN
-F 2 "" V 1580 4950 50  0000 C CNN
-F 3 "" H 1650 4950 50  0000 C CNN
-	1    1650 4950
-	1    0    0    -1
-$EndComp
-$Comp
-L R R?
-U 1 1 5806F0AD
-P 2300 4950
-F 0 "R?" V 2380 4950 50  0000 C CNN
-F 1 "R" V 2300 4950 50  0000 C CNN
-F 2 "" V 2230 4950 50  0000 C CNN
-F 3 "" H 2300 4950 50  0000 C CNN
-	1    2300 4950
-	1    0    0    -1
-$EndComp
-$Comp
-L C C?
-U 1 1 5806F2D0
-P 2100 4950
-F 0 "C?" H 2125 5050 50  0000 L CNN
-F 1 "C" H 2125 4850 50  0000 L CNN
-F 2 "" H 2138 4800 50  0000 C CNN
-F 3 "" H 2100 4950 50  0000 C CNN
-	1    2100 4950
-	-1   0    0    1
-$EndComp
-Text GLabel 2950 3950 2    60   Output ~ 0
+Text GLabel 2650 3950 2    60   Output ~ 0
 ALERT1
 Wire Wire Line
@@
 	1250 3800 1250 4450
 Wire Wire Line
-	2700 3800 2700 4450
-Wire Wire Line
-	2300 3800 2300 4800
-Wire Wire Line
-	2100 4700 2400 4700
-Wire Wire Line
-	1650 3800 1650 4800
-Wire Wire Line
-	1650 4700 1550 4700
-Wire Wire Line
-	1800 3950 1650 3950
-Connection ~ 1650 3950
-Wire Wire Line
-	2100 3950 2950 3950
-Connection ~ 2700 3950
-Wire Wire Line
-	2100 4200 2300 4200
-Connection ~ 2300 4200
-Wire Wire Line
-	1800 4200 1250 4200
-Connection ~ 1250 4200
-Wire Wire Line
-	1250 3350 1250 3500
-Wire Wire Line
-	1250 3350 2700 3350
-Wire Wire Line
-	2700 3350 2700 3500
-Wire Wire Line
-	2300 3500 2300 3350
-Connection ~ 2300 3350
-Wire Wire Line
-	1650 3500 1650 3350
-Connection ~ 1650 3350
-Connection ~ 1650 4700
-Connection ~ 2300 4700
-Wire Wire Line
-	2100 4800 2100 4700
-Wire Wire Line
-	2700 4850 2700 5200
-Wire Wire Line
-	2700 5200 1250 5200
-Wire Wire Line
-	1250 5200 1250 4850
-Wire Wire Line
-	1650 5100 1650 5200
-Connection ~ 1650 5200
-Wire Wire Line
-	2100 5100 2100 5200
-Connection ~ 2100 5200
-Wire Wire Line
-	2300 5100 2300 5200
-Connection ~ 2300 5200
+	2400 3800 2400 4450
+Wire Wire Line
+	1750 4700 1550 4700
+Connection ~ 2400 3950
+Wire Wire Line
+	1250 3400 1250 3500
+Wire Wire Line
+	2400 3400 2400 3500
 Text GLabel 1000 3950 0    60   Output ~ 0
 ALERT2
 Wire Wire Line
-	1000 3950 1250 3950
+	1000 3950 1350 3950
 Connection ~ 1250 3950
+Wire Wire Line
+	2300 3950 2650 3950
+Wire Wire Line
+	1650 3950 1750 3950
+Wire Wire Line
+	1750 3950 1750 4700
+Wire Wire Line
+	2300 4200 2400 4200
+Connection ~ 2400 4200
+Wire Wire Line
+	2000 3950 1900 3950
+Wire Wire Line
+	1900 3950 1900 4700
+Wire Wire Line
+	1900 4700 2100 4700
+Wire Wire Line
+	1350 4350 1250 4350
+Connection ~ 1250 4350
+Wire Wire Line
+	1650 4350 1900 4350
+Connection ~ 1900 4350
+Wire Wire Line
+	2000 4200 1750 4200
+Connection ~ 1750 4200
+Wire Wire Line
+	2400 4850 2400 4950
+Wire Wire Line
+	2400 4950 1250 4950
+Wire Wire Line
+	1250 4950 1250 4850
+Wire Wire Line
+	1250 3400 2400 3400
+Text GLabel 1750 6500 2    60   Input ~ 0
+ALERT
+$Comp
+L +24V_BJH #PWR?
+U 1 1 58161080
+P 3250 6300
+F 0 "#PWR?" H 3250 6490 20  0001 C CNN
+F 1 "+24V_BJH" H 3250 6490 51  0001 C CNN
+F 2 "" H 3250 6300 60  0001 C CNN
+F 3 "" H 3250 6300 60  0001 C CNN
+F 4 "+24V" H 3250 6500 60  0000 C CNB "NAME"
+	1    3250 6300
+	1    0    0    -1
+$EndComp
+$Comp
+L R R?
+U 1 1 581610E5
+P 1250 5900
+F 0 "R?" V 1330 5900 50  0000 C CNN
+F 1 "R" V 1250 5900 50  0000 C CNN
+F 2 "" V 1180 5900 50  0000 C CNN
+F 3 "" H 1250 5900 50  0000 C CNN
+	1    1250 5900
+	1    0    0    -1
+$EndComp
+Wire Wire Line
+	1250 5650 1250 5750
+Wire Wire Line
+	1250 6050 1250 6250
+Wire Wire Line
+	1750 6500 1550 6500
+Wire Wire Line
+	3250 6350 3250 6500
+Wire Wire Line
+	3250 6500 3500 6500
 $EndSCHEMATC

Commit message: Work on the ALERT signal
Parts:
- removed R?: R, symbol R
- added D? (x2): LED, symbol LED
- added J?: ALERT LED 1, symbol CONN_01X02
- added J?: ALERT LED 2, symbol CONN_01X02
- added Q? (x4): 2N7002, symbol 2N7002
- added R?: 1k5, symbol R
- added R? (x3): 10, symbol R
- C? (x2): value C -> 220n
- R? (x2): value R -> 10k
- R? (x2): value R -> 1M
Connections:
- net labels removed: ALERT
- wire segments 50 -> 73
