File: Hardware/KiCAD/Power.sch (KiCad schematic (older format))
At the start: 0 parts

Commit message: more work on the schematic
Parts:
- added C?: 10uF, symbol CP1
- added C? (x4): 0.1uF, symbol C
- added C?: 1uF, symbol C
- added C?: 0.01uF, symbol C
- added C?: CP1, symbol CP1
- added D?: D, symbol D
- added R?: R, symbol R
- added U?: PIC18F25K80, symbol PIC18F25K80
- added U?: RN4020, symbol RN4020
- added U?: POXA1328-007, symbol POXA1328-007
- added U?: S25FL127S_SOIC, symbol S25FL127S_SOIC
- added U?: MCP795XX, symbol MCP795XX
Connections:
- net labels added: +3.3V_BJH, GND
- wire segments 0 -> 45
Other:
- note added: "(must use low ESR)"

Commit message: more work on PTWS schematic
Parts:
- added C10, C13, C15, C17, C18, C23, C24, C9: 0.1uF, symbol C
- added C16: C, symbol C
- added R10: 1K, symbol R
- added U5, U6: 4000series-4052, DIP16, symbol 4000series-4052
- added U8, U9: MAX3232_BJH, maxim-DIL16, symbol MAX3232_BJH
- D1: renamed from D?; value D -> DB27308
- R9: renamed from R?; value R -> 30R
- U4: renamed from U?; symbol S25FL127S_SOIC -> S25FL127S_SOIC-RESCUE-ptws
- gave numbers to parts that had none: 12
Connections:
- net labels added: +24V_BJH, VBAT_BJH
- wire segments 45 -> 83
Other:
- moved on the sheet: C11, D1, R9

Commit message: More work on PTWS schematic
Connections:
- net +3.3V: no longer U2.4 (VBK)
- no-connect marks 0 -> 1
Changed lines of the file:
@@
 	3850 1950 3850 2550
 Connection ~ 3850 2550
-Wire Wire Line
-	4650 1000 4650 1300
 Connection ~ 4450 1000
 Wire Wire Line
 	5050 1000 5050 1650
-Connection ~ 4650 1000
 Wire Wire Line
 	5050 2550 5050 1950
@@
 EndData
 $EndBitmap
+NoConn ~ 4650 1300
 $EndSCHEMATC
